File: Pi-880Backplane.brd (EAGLE design)
At the start: 105.4 x 71.1 mm, 2 parts

Commit message: First board
Routing:
- net N$6: track 0.00 -> 7.62 mm
- net N$2: track 0.00 -> 7.62 mm
- net N$16: track 0.00 -> 7.62 mm
- net N$13: track 0.00 -> 7.62 mm
- net N$12: track 0.00 -> 7.62 mm
- net N$11: track 0.00 -> 7.62 mm
- net N$3: track 0.00 -> 7.62 mm
- net N$14: track 0.00 -> 7.62 mm
- net N$10: track 0.00 -> 7.62 mm
- net N$1: track 0.00 -> 7.62 mm
- net N$9: track 0.00 -> 7.62 mm
- net N$8: track 0.00 -> 7.62 mm
- net N$4: track 0.00 -> 7.62 mm
- net N$15: track 0.00 -> 7.62 mm
- net N$7: track 0.00 -> 7.62 mm
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Changed lines of the file:
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@@
 <hole x="99.06" y="38.1" drill="5.5"/>
 <text x="90.17" y="55.88" size="1.778" layer="16" rot="MR0">v1, 10.1.16, Tobias Cottmann</text>
+<circle x="-5.08" y="71.12" radius="2.54" width="0.254" layer="16"/>
+<circle x="-5.08" y="0" radius="2.54" width="0.254" layer="16"/>
+<circle x="110.49" y="71.12" radius="2.54" width="0.254" layer="16"/>
+<circle x="110.49" y="0" radius="2.54" width="0.254" layer="16"/>
+<circle x="0" y="-5.08" radius="2.54" width="0.254" layer="16"/>
+<circle x="105.41" y="76.2" radius="2.54" width="0.254" layer="16"/>
+<circle x="105.41" y="-5.08" radius="2.54" width="0.254" layer="16"/>
+<circle x="0" y="76.2" radius="2.54" width="0.254" layer="16"/>
 </plain>
 <attributes>
@@
 <wire x1="58.42" y1="3.81" x2="60.96" y2="6.35" width="0.4064" layer="16"/>
 </signal>
+<signal name="N$1">
+<wire x1="-8.89" y1="71.12" x2="-1.27" y2="71.12" width="0.254" layer="16"/>
+</signal>
+<signal name="N$2">
+<wire x1="-5.08" y1="74.93" x2="-5.08" y2="67.31" width="0.254" layer="16"/>
+</signal>
+<signal name="N$3">
+<wire x1="-8.89" y1="0" x2="-1.27" y2="0" width="0.254" layer="16"/>
+</signal>
+<signal name="N$4">
+<wire x1="-5.08" y1="3.81" x2="-5.08" y2="-3.81" width="0.254" layer="16"/>
+</signal>
+<signal name="N$5">
+<wire x1="106.68" y1="71.12" x2="114.3" y2="71.12" width="0.254" layer="16"/>
+</signal>
+<signal name="N$6">
+<wire x1="110.49" y1="74.93" x2="110.49" y2="67.31" width="0.254" layer="16"/>
+</signal>
+<signal name="N$7">
+<wire x1="106.68" y1="0" x2="114.3" y2="0" width="0.254" layer="16"/>
+</signal>
+<signal name="N$8">
+<wire x1="110.49" y1="3.81" x2="110.49" y2="-3.81" width="0.254" layer="16"/>
+</signal>
+<signal name="N$9">
+<wire x1="-3.81" y1="-5.08" x2="3.81" y2="-5.08" width="0.254" layer="16"/>
+</signal>
+<signal name="N$10">
+<wire x1="0" y1="-1.27" x2="0" y2="-8.89" width="0.254" layer="16"/>
+</signal>
+<signal name="N$11">
+<wire x1="101.6" y1="76.2" x2="109.22" y2="76.2" width="0.254" layer="16"/>
+</signal>
+<signal name="N$12">
+<wire x1="105.41" y1="80.01" x2="105.41" y2="72.39" width="0.254" layer="16"/>
+</signal>
+<signal name="N$13">
+<wire x1="101.6" y1="-5.08" x2="109.22" y2="-5.08" width="0.254" layer="16"/>
+</signal>
+<signal name="N$14">
+<wire x1="105.41" y1="-1.27" x2="105.41" y2="-8.89" width="0.254" layer="16"/>
+</signal>
+<signal name="N$15">
+<wire x1="-3.81" y1="76.2" x2="3.81" y2="76.2" width="0.254" layer="16"/>
+</signal>
+<signal name="N$16">
+<wire x1="0" y1="80.01" x2="0" y2="72.39" width="0.254" layer="16"/>
+</signal>
 </signals>

Commit message: Merged v2
Parts:
- added U$3: SMA-PIGTAIL-MOUNT, tobias:SMA-PIGTAIL-MOUNT
- added X1: (no value), con-phoenix-254:2POL254
- U$1: value RPI-ZERO -> RPI-ZERONODRILLS; device RPI-Zero:RASPBERRYPI_BASTELSTUBE_V13_RASPI_BOARD_B+_FULL -> tobias:RPI-ZERO-NODRILLS
- moved U$1 55.9 mm to (36.8, 67.3), flipped to the bottom
- moved U$2 24.3 mm to (-12.7, 0.00)
Connections:
- net GND: now also U$3.GND, X1.2
- net VCC: now also X1.1
Routing:
- net SPI_CLK: track 88.5 -> 37.2 mm
- net NSS: track 108.5 -> 57.4 mm
- net MOSI: track 76.9 -> 44.4 mm
- net MISO: track 72.5 -> 40.8 mm
- net RESET: track 63.9 -> 42.1 mm
- net VCC: track 24.6 -> 12.7 mm
- net N$6: track 7.62 -> 0.00 mm
- net N$2: track 7.62 -> 0.00 mm
- net N$16: track 7.62 -> 0.00 mm
- net N$13: track 7.62 -> 0.00 mm
- net N$12: track 7.62 -> 0.00 mm
- net N$11: track 7.62 -> 0.00 mm
- net N$3: track 7.62 -> 0.00 mm
- net N$14: track 7.62 -> 0.00 mm
- net N$10: track 7.62 -> 0.00 mm
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- added copper zone on layer 1, net GND
Other:
- board size 105.4 x 71.1 mm -> 57.1 x 80 mm
- board text removed: "v1, 10.1.16, Tobias Cottmann"
